File: device/hw/foodSampler_v10/foodSampler_v10.kicad_pcb (KiCad board)
At the start: 2 copper layers, 70 x 128 mm, 50 parts, among them J00 Conn_01x16, J01 Conn_01x12, Q00 BSS138, SW10 SWITCH_SPST_LED, SW20 SWITCH_SPST_LED, SW30 SWITCH_SPST_LED, SW40 SWITCH_SPST_LED, SW50 SWITCH_SPST_LED, SW60 SWITCH_SPST_LED, SW70 SWITCH_SPST_LED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

Commit message: to compare
Parts:
- REF**: moved to B.Cu
- turned REF** to 270 degrees
Changed lines of the file:
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@@
   (page A4)
   (layers
-    (0 F.Cu signal)
-    (31 B.Cu signal)
-    (32 B.Adhes user)
-    (33 F.Adhes user)
+    (0 F.Cu signal hide)
+    (31 B.Cu signal hide)
+    (32 B.Adhes user hide)
+    (33 F.Adhes user hide)
     (34 B.Paste user)
     (35 F.Paste user)
@@
     (pad "" np_thru_hole circle (at 0 -4.5) (size 1.8 1.8) (drill 1.7) (layers *.Cu *.Mask))
   )
-  (module _special:LIPO_3V7_2A_50x60 (layer F.Cu)
-    (at 89.9 76.2 90)
+  (module _special:LIPO_3V7_2A_50x60 (layer B.Cu)
+    (at 89.9 76.2 270)
     (tags "lipo, battery")
-    (fp_text reference REF** (at 12 -28 90) (layer F.SilkS) hide
-      (effects (font (size 1 1) (thickness 0.15)))
-    )
-    (fp_text value LIPO_3V7_2A_50x60 (at 17 -26 90) (layer F.Fab)
-      (effects (font (size 1 1) (thickness 0.15)))
-    )
-    (fp_line (start -25 -20) (end 25 -20) (layer F.CrtYd) (width 0.15))
-    (fp_line (start -25 -30) (end 0 -30) (layer F.CrtYd) (width 0.15))
-    (fp_line (start -25 30) (end -25 -30) (layer F.CrtYd) (width 0.15))
-    (fp_line (start 25 30) (end -25 30) (layer F.CrtYd) (width 0.15))
-    (fp_line (start 25 -30) (end 25 30) (layer F.CrtYd) (width 0.15))
-    (fp_line (start 0 -30) (end 25 -30) (layer F.CrtYd) (width 0.15))
+    (fp_text reference REF** (at 12 28 270) (layer B.SilkS) hide
+      (effects (font (size 1 1) (thickness 0.15)) (justify mirror))
+    )
+    (fp_text value LIPO_3V7_2A_50x60 (at 17 26 270) (layer B.Fab)
+      (effects (font (size 1 1) (thickness 0.15)) (justify mirror))
+    )
+    (fp_line (start -25 20) (end 25 20) (layer B.CrtYd) (width 0.15))
+    (fp_line (start -25 30) (end 0 30) (layer B.CrtYd) (width 0.15))
+    (fp_line (start -25 -30) (end -25 30) (layer B.CrtYd) (width 0.15))
+    (fp_line (start 25 -30) (end -25 -30) (layer B.CrtYd) (width 0.15))
+    (fp_line (start 25 30) (end 25 -30) (layer B.CrtYd) (width 0.15))
+    (fp_line (start 0 30) (end 25 30) (layer B.CrtYd) (width 0.15))
   )
   (module Connector_PinHeader_2.54mm:PinHeader_1x12_P2.54mm_Vertical_SMD_Pin1Left (layer B.Cu)
