File: device/hw/foodSampler_v21/foodSampler_v21.kicad_pcb (KiCad board)
At the start: 2 copper layers, 162 x 128 mm, 86 parts, among them J00 USB_C_Receptacle, J20 BATT1, Q10 MMBT3904, Q11 MMBT3904, SW00 SWITCH_SPDT, SW10 NO, SW11 NO, SW40 SWITCH_LED, SW41 SWITCH_LED, SW42 SWITCH_LED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

Commit message: _sampler V2.2 added
Connections:
- RS44 pad 2: Net-(RS44-Pad2) -> SW4
Routing:
- net VOUT: track 62.4 -> 66.7 mm
- net VBUS: track 37.1 -> 38.0 mm
- net GND: vias 40 -> 46
Other:
- board text added: "_sampler V2.1 210517MCH"
- board text removed: "FoodSampler V2.1 210517MCH"
