File: device/hw/foodSampler_v21/foodSampler_v21.sch (KiCad schematic (older format))
At the start: 80 parts, among them J00 USB_C_Receptacle, J20 BATT1, Q10 MMBT3904, Q11 MMBT3904, SW00 SWITCH_SPDT, SW10 NO, SW11 NO, SW40 SWITCH_LED, SW41 SWITCH_LED, SW42 SWITCH_LED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

Commit message: _sampler V2.2 added
Connections:
- net SW4: now also RS44.2
Changed lines of the file:
@@
 	3500 10300 3500 10250
 Connection ~ 3500 10250
+Wire Wire Line
+	1900 9900 2150 9900
+Connection ~ 2150 9900
 $EndSCHEMATC
