File: device/hw/foodSampler_v22/foodSampler_v22.sch (KiCad schematic (older format))
At the start: 94 parts, among them J00 USB_C_Receptacle, J20 BATT1, Q10 MMBT3904, Q11 MMBT3904, SW00 SWITCH_SPDT, SW10 NO, SW11 NO, SW40 SWITCH_LED, SW41 SWITCH_LED, SW42 SWITCH_LED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

Commit message: small revisions
Parts:
- C11: value 100nF -> 10uF
- C30: value 470pF -> 22pF
- C31: value 2.2uF -> 10uF
Changed lines of the file:
@@
 P 8200 7150
 F 0 "C11" H 8150 6950 50  0000 L CNN
-F 1 "100nF" H 8100 6850 50  0000 L CNN
+F 1 "10uF" H 8100 6850 50  0000 L CNN
 F 2 "Capacitor_SMD:C_0603_1608Metric" H 8200 7150 50  0001 C CNN
 F 3 "~" H 8200 7150 50  0001 C CNN
@@
 P 10900 1850
 F 0 "C30" H 10992 1896 50  0000 L CNN
-F 1 "470pF" H 10992 1805 50  0000 L CNN
+F 1 "22pF" H 10992 1805 50  0000 L CNN
 F 2 "Capacitor_SMD:C_0603_1608Metric" H 10900 1850 50  0001 C CNN
 F 3 "~" H 10900 1850 50  0001 C CNN
@@
 P 11300 1850
 F 0 "C31" H 11392 1896 50  0000 L CNN
-F 1 "2.2uF" H 11400 1800 50  0000 L CNN
+F 1 "10uF" H 11400 1800 50  0000 L CNN
 F 2 "Capacitor_Tantalum_SMD:CP_EIA-3216-10_Kemet-I" H 11300 1850 50  0001 C CNN
 F 3 "~" H 11300 1850 50  0001 C CNN
